Commit message: cleaning robot controller tuning and giraffe microphone orientation fixes

File: src/giraffe_robot/urdf/giraffe.urdf (robot description, URDF)
Before this commit: robot giraffe_robot, 8 links, 7 joints
Joints:
- removed joint joint5_roll
- added joint joint5_yaw: type revolute, parent link4_wrist, child end_effector, origin xyz=0 0 0 rpy=0 0 0, axis 0 0 1, limit lower=-3.14 upper=3.14 effort=50 velocity=2.0
- joint joint_mic_tip: origin xyz=0 0 0.10 rpy=0 0 0 -> xyz=-0.10 0 0.2 rpy=0 0 0
