Commit message: cleaning robot

File: src/cleaning_robot/urdf/assembly.urdf (robot description, URDF)
Before this commit: robot cleaning_robot, 14 links, 13 joints
Joints:
- joint tool_tip_fixed: origin xyz=0.03 0 0 rpy=0 1.5708 0 -> xyz=0.03 0 0 rpy=3.14159 0 0

File: src/giraffe_robot/urdf/giraffe.urdf (robot description, URDF)
Before this commit: robot giraffe_robot, 7 links, 6 joints
Links:
- added link mic_tip, mass 0.01; visual sphere radius=0.015
- link end_effector: geometry visual cylinder length=0.1 radius=0.01
Joints:
- added joint joint_mic_tip: type fixed, parent end_effector, child mic_tip, origin xyz=0 0 0.10 rpy=0 0 0
- joint joint1_pan: limit lower=-3.14 upper=3.14 effort=100 velocity=1.0 -> lower=-3.14 upper=3.14 effort=200 velocity=2.0
- joint joint2_tilt: limit lower=-1.57 upper=0.0 effort=100 velocity=1.0 -> lower=-1.57 upper=0.0 effort=200 velocity=2.0
- joint joint3_prismatic: limit lower=0.0 upper=7.0 effort=200 velocity=2 -> lower=0.0 upper=7.0 effort=400 velocity=1

Commit message: fix

File: src/cleaning_robot/urdf/assembly.urdf (robot description, URDF)
Before this commit: robot cleaning_robot, 14 links, 13 joints
Joints:
- joint z1_joint2: limit lower=-2.094 upper=2.094 effort=33.5 velocity=3.14 -> lower=-2.094 upper=2.094 effort=60 velocity=3.14
